File: project_files/highway_wave/highway_wave.kicad_sch (KiCad schematic)
At the start: 8 parts, among them J1 Screw_Terminal_01x02, J2 Screw_Terminal_01x02, J3 Conn_01x02_Socket, J4 Conn_01x02_Socket, J8 Conn_01x04_Socket, U1 GW1N-LV9QN88C6_I5_, U2 MOUDLE-BLUETOOTH-AUDIO-BC127_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, U4 PAM8403D

Commit message: fixed pcb
Parts:
- removed U1: GW1N-LV9QN88C6_I5_, GW1N-LV9QN88C6_I5_:QFN40P1000X1000X95-89N, symbol GW1N-LV9QN88C6_I5_:GW1N-LV9QN88C6_I5_
- added C10: 47 uF, Capacitor_THT:CP_Radial_D5.0mm_P2.50mm, symbol Device:C_Polarized_US
- added C9: 1 uF, Capacitor_THT:CP_Radial_D5.0mm_P2.50mm, symbol Device:C
- added J10: Conn_01x02_Socket, Connector_JST:JST_PH_B2B-PH-K_1x02_P2.00mm_Vertical, symbol Connector:Conn_01x02_Socket
- added J11, J12: Conn_01x24, Connector_PinSocket_2.54mm:PinSocket_1x24_P2.54mm_Vertical, symbol Connector_Generic:Conn_01x24
- added J13: Screw_Terminal_01x02, TerminalBlock_MetzConnect:TerminalBlock_MetzConnect_Type101_RT01602HBWC_1x02_P5.08mm_Horizontal, symbol Connector:Screw_Terminal_01x02
- added U1: TPS75633KC, footprints:KC5, symbol Battery Regulator:TPS75633KC
- J3, J4: footprint Connector_Phoenix_GMSTB:PhoenixContact_GMSTBVA_2,5_2-G_1x02_P7.50mm_Vertical -> Connector_JST:JST_PH_B2B-PH-K_1x02_P2.00mm_Vertical
- J8: footprint Connector_Phoenix_GMSTB:PhoenixContact_GMSTBVA_2,5_4-G_1x04_P7.50mm_Vertical -> Connector_JST:JST_PH_B2B-PH-K_1x02_P2.00mm_Vertical
Connections:
- net 28_IOB11B: now reaches U2.41 (UART-TX)
- net 28_IOB11B: now also J12.8 (Pin_8)
- net 27_IOB11A: now reaches U2.42 (UART-RX)
- net 27_IOB11A: now also J12.7 (Pin_7)
- net 30_IOB13B: now reaches U4.7 (INL)
- net 30_IOB13B: now also J12.10 (Pin_10)
- net 29_IOB13A: now reaches U4.10 (INR)
- net 29_IOB13A: now also J12.9 (Pin_9)
- net +3V3 renamed IN_3V3
- net IN_3V3: now also C9.2, J10.1 (Pin_1), J13.1 (Pin_1), U1.1 (EN), U1.2 (IN); no longer U2.34 (3V3-USB)
- net GND renamed IN_GND
- net IN_GND: now also C10.2, C9.1, J10.2 (Pin_2), J11.23 (Pin_23), J13.2 (Pin_2), U1.3 (GND)
- net TDM CLK renamed 36_IOB29B
- net 36_IOB29B: now also J12.3 (Pin_3)
- net TDM SD renamed 26_IOB8B
- net 26_IOB8B: now also J12.6 (Pin_6)
- net TDM WS renamed 25_IOB8A
- net 25_IOB8A: now also J12.5 (Pin_5)
- net VCC renamed Vout from Bat reg
- net Vout from Bat reg: now also U2.34 (3V3-USB), C10.1, J11.24 (Pin_24), U1.4 (OUTPUT)
- new net 31_IOB15A: J11.21 (Pin_21)
- new net 32_IOB15B: J11.22 (Pin_22)
- new net 33_IOB23A: J12.11 (Pin_11)
- new net 34_IOB23B: J12.12 (Pin_12)
- new net 35_IOB29A: J12.14 (Pin_14)
- new net 37_IOB31A: J12.2 (Pin_2)
- new net 38_IOB31B: J12.1 (Pin_1)
- new net 39_IOB33A: J12.4 (Pin_4)
- new net 40_IOB33B: J12.13 (Pin_13)
- new net 41_IOB41A: J12.15 (Pin_15)
- new net 42_IOB41B: J12.16 (Pin_16)
- new net 48_IOR24B: J11.19 (Pin_19)
- new net 49_IOR24B: J11.20 (Pin_20)
- new net 51_IOR17B: J12.17 (Pin_17)
- new net 53_IOR15B: J12.18 (Pin_18)
- new net 54_IOR15A: J12.19 (Pin_19)
- new net 55_IOR14B: J12.20 (Pin_20)
- new net 56_IOR14A: J12.21 (Pin_21)
- new net 57_IOR13A: J12.22 (Pin_22)
- new net 63_IOR5A: J11.1 (Pin_1)
- new net 68_IOT42B: J12.23 (Pin_23)
- new net 69_IOT42A: J12.24 (Pin_24)
- new net 70_IOT41B: J11.17 (Pin_17)
- new net 71_IOT41A: J11.16 (Pin_16)
- new net 72_IOT39B: J11.15 (Pin_15)
- new net 73_IOT39A: J11.14 (Pin_14)
- new net 74_IOT38B: J11.13 (Pin_13)
- new net 75_IOT38A: J11.12 (Pin_12)
- new net 76_IOT37B: J11.11 (Pin_11)
- new net 77_IOT37A: J11.10 (Pin_10)
- new net 79_IOT12B: J11.9 (Pin_9)
- new net 80_IOT12A: J11.8 (Pin_8)
- new net 81_IOT11B: J11.7 (Pin_7)
- new net 82_IOT11A: J11.6 (Pin_6)
- new net 83_IOT10B: J11.5 (Pin_5)
- new net 84_IOT10A: J11.4 (Pin_4)
- new net 85_IOT8B: J11.3 (Pin_3)
- new net 86_IOT8A: J11.2 (Pin_2)
- new net IN_5V: J11.18 (Pin_18)
Other:
- moved on the sheet: J1, J2, J3, J4, J8, U2, U4

Commit message: update BOM
Parts:
- removed C10: 47 uF, Capacitor_THT:CP_Radial_D5.0mm_P2.50mm, symbol Device:C_Polarized_US
- removed C9: 1 uF, Capacitor_THT:CP_Radial_D5.0mm_P2.50mm, symbol Device:C
- removed J4: Conn_01x02_Socket, Connector_JST:JST_PH_B2B-PH-K_1x02_P2.00mm_Vertical, symbol Connector:Conn_01x02_Socket
- removed J8: Conn_01x04_Socket, Connector_JST:JST_PH_B2B-PH-K_1x02_P2.00mm_Vertical, symbol Connector:Conn_01x04_Socket
- removed U1: TPS75633KC, footprints:KC5, symbol Battery Regulator:TPS75633KC
- removed U2: MOUDLE-BLUETOOTH-AUDIO-BC127_51P-18X11.8MM_, MOUDLE-BLUETOOTH-AUDIO-BC127_51P-18X11.8MM_:LGA51-0.8-18X11.8MM, symbol MOUDLE-BLUETOOTH-AUDIO-BC127_51P-18X11.8MM_:MOUDLE-BLUETOOTH-AUDIO-BC127_51P-18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
- removed U4: PAM8403D, Package_SO:SOP-16_3.9x9.9mm_P1.27mm, symbol Amplifier_Audio:PAM8403D
- added J11, J12, J14, J15, J16, J17, J18, J19, J22, J23, J24, J25, J7, J9: Conn_01x02_Socket, Connector_JST:JST_PH_B2B-PH-K_1x02_P2.00mm_Vertical, symbol Connector:Conn_01x02_Socket
- renumbered J12 to J1, J11 to J2, J1 to J20, J2 to J21, J10 to J5
Connections:
- net Vout from Bat reg is gone; now on net 69_IOT42A: J2.24 (Pin_24)
- net 25_IOB8A: now also J2.5 (Pin_5), J7.1 (Pin_1); no longer J1.5 (Pin_5)
- net 26_IOB8B: now also J2.6 (Pin_6); no longer J1.6 (Pin_6)
- net 27_IOB11A: now also J2.7 (Pin_7); no longer J1.7 (Pin_7)
- net 28_IOB11B: now also J2.8 (Pin_8); no longer J1.8 (Pin_8)
- net 29_IOB13A: now also J2.9 (Pin_9), J12.1 (Pin_1), J22.1 (Pin_1); no longer J1.9 (Pin_9)
- net 30_IOB13B: now also J2.10 (Pin_10), J12.2 (Pin_2), J22.2 (Pin_2); no longer J1.10 (Pin_10)
- net 31_IOB15A: now also J1.21 (Pin_21); no longer J2.21 (Pin_21)
- net 32_IOB15B: now also J1.22 (Pin_22); no longer J2.22 (Pin_22)
- net 33_IOB23A: now also J2.11 (Pin_11); no longer J1.11 (Pin_11)
- net 34_IOB23B: now also J2.12 (Pin_12); no longer J1.12 (Pin_12)
- net 35_IOB29A: now also J2.14 (Pin_14); no longer J1.14 (Pin_14)
- net 36_IOB29B: now also J2.3 (Pin_3); no longer J1.3 (Pin_3)
- net 37_IOB31A: now also J2.2 (Pin_2); no longer J1.2 (Pin_2)
- net 38_IOB31B: now also J2.1 (Pin_1); no longer J1.1 (Pin_1)
- net 39_IOB33A: now also J2.4 (Pin_4); no longer J1.4 (Pin_4)
- net 40_IOB33B: now also J2.13 (Pin_13); no longer J1.13 (Pin_13)
- net 41_IOB41A: now also J2.15 (Pin_15); no longer J1.15 (Pin_15)
- net 42_IOB41B: now also J2.16 (Pin_16); no longer J1.16 (Pin_16)
- net 48_IOR24B: now also J1.19 (Pin_19); no longer J2.19 (Pin_19)
- net 49_IOR24B: now also J1.20 (Pin_20); no longer J2.20 (Pin_20)
- net 51_IOR17B: now also J2.17 (Pin_17); no longer J1.17 (Pin_17)
- net 53_IOR15B: now also J2.18 (Pin_18); no longer J1.18 (Pin_18)
- net 54_IOR15A: now also J2.19 (Pin_19); no longer J1.19 (Pin_19)
- net 55_IOR14B: now also J2.20 (Pin_20); no longer J1.20 (Pin_20)
- net 56_IOR14A: now also J2.21 (Pin_21); no longer J1.21 (Pin_21)
- net 57_IOR13A: now also J2.22 (Pin_22); no longer J1.22 (Pin_22)
- net 63_IOR5A: now also J1.1 (Pin_1); no longer J2.1 (Pin_1)
- net 68_IOT42B: now also J2.23 (Pin_23); no longer J1.23 (Pin_23)
- net 69_IOT42A: no longer J1.24 (Pin_24)
- net 70_IOT41B: now also J1.17 (Pin_17); no longer J2.17 (Pin_17)
- net 71_IOT41A: now also J1.16 (Pin_16); no longer J2.16 (Pin_16)
- net 72_IOT39B: now also J1.15 (Pin_15); no longer J2.15 (Pin_15)
- net 73_IOT39A: now also J1.14 (Pin_14); no longer J2.14 (Pin_14)
- net 74_IOT38B: now also J1.13 (Pin_13); no longer J2.13 (Pin_13)
- net 75_IOT38A: now also J1.12 (Pin_12); no longer J2.12 (Pin_12)
- net 76_IOT37B: now also J1.11 (Pin_11); no longer J2.11 (Pin_11)
- net 77_IOT37A: now also J1.10 (Pin_10); no longer J2.10 (Pin_10)
- net 79_IOT12B: now also J1.9 (Pin_9); no longer J2.9 (Pin_9)
- net 80_IOT12A: now also J1.8 (Pin_8); no longer J2.8 (Pin_8)
- net 81_IOT11B: now also J1.7 (Pin_7); no longer J2.7 (Pin_7)
- net 82_IOT11A: now also J1.6 (Pin_6); no longer J2.6 (Pin_6)
- net 83_IOT10B: now also J1.5 (Pin_5); no longer J2.5 (Pin_5)
- net 84_IOT10A: now also J1.4 (Pin_4); no longer J2.4 (Pin_4)
- net 85_IOT8B: now also J1.3 (Pin_3); no longer J2.3 (Pin_3)
- net 86_IOT8A: now also J1.2 (Pin_2); no longer J2.2 (Pin_2)
- net IN_3V3: now also J1.24 (Pin_24), J11.1 (Pin_1), J14.1 (Pin_1), J15.1 (Pin_1), J19.1 (Pin_1)
- net IN_5V: now also J1.18 (Pin_18); no longer J2.18 (Pin_18)
- net IN_GND: now also J1.23 (Pin_23), J11.2 (Pin_2), J14.2 (Pin_2), J15.2 (Pin_2), J16.1 (Pin_1), J16.2 (Pin_2), J19.2 (Pin_2), J23.1 (Pin_1), J23.2 (Pin_2); no longer J2.23 (Pin_23)
- net LOUT+: now reaches J20.1 (Pin_1)
- net LOUT+: now also J17.1 (Pin_1)
- net headphone_ROUT+: now reaches J21.1 (Pin_1)
- net headphone_ROUT+: now also J24.1 (Pin_1)
- net headphone_ROUT-: now reaches J21.2 (Pin_2)
- net headphone_ROUT-: now also J24.2 (Pin_2)
- net LOUT-: now reaches J20.2 (Pin_2)
- net LOUT-: now also J17.2 (Pin_2)
- new net: J7.2 (Pin_2), J9.2 (Pin_2)
- new net ROUT+: J18.1 (Pin_1), J25.1 (Pin_1)
- new net ROUT-: J18.2 (Pin_2), J25.2 (Pin_2)
Other:
- note added: "BLE"
- note added: "batt for amp"
- note added: "extra in case LiPo is JST"
- note added: "left input"
- note added: "right input"
- note added: "to charge reg"
- moved on the sheet: J1, J13, J2, J20, J21, J3, J5
