File: project_files/highway_wave/untitled.kicad_sch (KiCad schematic)
At the start: 17 parts

Commit message: random committ
Parts:
- added J5, J6, J7, J9: Conn_01x02_Pin, Connector_Phoenix_GMSTB:PhoenixContact_GMSTBVA_2,5_2-G_1x02_P7.50mm_Vertical, symbol Connector:Conn_01x02_Pin
- added R2: 100 k, Resistor_THT:R_Axial_DIN0207_L6.3mm_D2.5mm_P7.62mm_Horizontal, symbol Device:R
Connections:
- net GND: now also R1.1; no longer C5.2, C6.2, C7.2, C8.2, MK5.4_1 (GND), MK5.4_2 (GND), MK5.4_3 (GND), MK5.4_4 (GND), MK6.4_1 (GND), MK6.4_2 (GND), MK6.4_3 (GND), MK6.4_4 (GND), MK7.4_1 (GND), MK7.4_2 (GND), MK7.4_3 (GND), MK7.4_4 (GND), MK8.4_1 (GND), MK8.4_2 (GND), MK8.4_3 (GND), MK8.4_4 (GND), R1.2
- net TDM CLK: no longer MK5.6 (SCK), MK6.6 (SCK), MK7.6 (SCK), MK8.6 (SCK)
- net TDM SD: now also R1.2; no longer MK5.7 (SD), MK6.7 (SD), MK7.7 (SD), MK8.7 (SD), R1.1
- net WSO Mk6: no longer MK7.5 (WS)
- net WSO Mk7: no longer MK7.1 (WSO), MK8.5 (WS)
- net TDM WS: no longer names the net of MK1.5 (WS)
- net TDM WS: now also J5.2 (Pin_2)
- net VCC: no longer names the net of C5.1, C6.1, C7.1, C8.1, MK5.2 (CONFIG), MK5.3 (VDD), MK6.2 (CONFIG), MK6.3 (VDD), MK7.2 (CONFIG), MK7.3 (VDD), MK8.2 (CONFIG), MK8.3 (VDD)
- net VCC: now also J7.1 (Pin_1); no longer C1.1, C2.1, C3.1, C4.1, MK1.2 (CONFIG), MK1.3 (VDD), MK2.2 (CONFIG), MK2.3 (VDD), MK3.2 (CONFIG), MK3.3 (VDD), MK4.2 (CONFIG), MK4.3 (VDD)
- net WSO Mk4: no longer names the net of MK5.5 (WS)
- net WSO Mk4: now also J9.1 (Pin_1), J9.2 (Pin_2); no longer MK4.1 (WSO)
- new net: C5.2, C6.2, C7.2, C8.2, J7.2 (Pin_2), MK5.4_1 (GND), MK5.4_2 (GND), MK5.4_3 (GND), MK5.4_4 (GND), MK6.4_1 (GND), MK6.4_2 (GND), MK6.4_3 (GND), MK6.4_4 (GND), MK7.4_1 (GND), MK7.4_2 (GND), MK7.4_3 (GND), MK7.4_4 (GND), MK8.4_1 (GND), MK8.4_2 (GND), MK8.4_3 (GND), MK8.4_4 (GND), R2.1
- new net: J6.1 (Pin_1), MK5.7 (SD), MK6.7 (SD), MK7.7 (SD), MK8.7 (SD), R2.2
- new net: J6.2 (Pin_2), MK5.6 (SCK), MK6.6 (SCK), MK7.6 (SCK), MK8.6 (SCK)
- new net: J5.1 (Pin_1), MK4.1 (WSO)
- new net +3V3: C1.1, C2.1, C3.1, C4.1, MK1.2 (CONFIG), MK1.3 (VDD), MK2.2 (CONFIG), MK2.3 (VDD), MK3.2 (CONFIG), MK3.3 (VDD), MK4.2 (CONFIG), MK4.3 (VDD)
Other:
- moved on the sheet: C1, C2, C3, C4, MK1, MK2, MK3, MK4, R1

Commit message: fixed pcb
Parts:
- C1, C2, C3, C4, C5, C6, C7, C8: footprint Capacitor_THT:CP_Radial_D8.0mm_P5.00mm -> Capacitor_THT:CP_Radial_D5.0mm_P2.50mm
- J5, J6, J7, J9: footprint Connector_Phoenix_GMSTB:PhoenixContact_GMSTBVA_2,5_2-G_1x02_P7.50mm_Vertical -> Connector_JST:JST_PH_B2B-PH-K_1x02_P2.00mm_Vertical
Connections:
- net +3V3 renamed Vout from Bat reg
- net GND renamed IN_GND
Other:
- moved on the sheet: C1, C2, C3, C4, C5, C6, C7, C8, J5, J6, J7, J9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

Commit message: update BOM
Parts:
- C1, C2, C3, C4, C5, C6, C7, C8: footprint Capacitor_THT:CP_Radial_D5.0mm_P2.50mm -> Capacitor_THT:C_Disc_D5.0mm_W2.5mm_P5.00mm
- renumbered J9 to J10, J6 to J4, J7 to J6, J5 to J8
Connections:
- net WSO Mk6: now also MK7.5 (WS)
- net WSO Mk7: now also MK7.1 (WSO), MK8.5 (WS)
- net Vout from Bat reg renamed IN_3V3
Changed lines of the file:
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@@
+		)
+	)
+	(global_label "IN_3V3"
+		(shape input)
+		(at 95.25 40.64 90)
+		(fields_autoplaced yes)
+		(effects
+			(font
+				(size 1.27 1.27)
+			)
+			(justify left)
+		)
+		(property "Intersheetrefs" "${INTERSHEET_REFS}"
+			(at 95.25 31.2443 90)
+			(effects
+				(font
+					(size 1.27 1.27)
+				)
+				(justify left)
+				(hide yes)
+			)
 		)
 	)
@@
 	(global_label "WSO Mk7"
 		(shape bidirectional)
-		(at 171.45 121.92 0)
+		(at 171.45 120.65 0)
 		(fields_autoplaced yes)
 		(effects
@@
 		)
 		(property "Intersheetrefs" "${INTERSHEET_REFS}"
-			(at 184.1945 121.92 0)
+			(at 184.1945 120.65 0)
 			(effects
 				(font
@@
 	(global_label "WSO Mk6"
 		(shape bidirectional)
-		(at 135.89 119.38 180)
+		(at 135.89 118.11 180)
 		(fields_autoplaced yes)
 		(effects
@@
 		)
 		(property "Intersheetrefs" "${INTERSHEET_REFS}"
-			(at 123.1455 119.38 0)
+			(at 123.1455 118.11 0)
 			(effects
 				(font
@@
 	(global_label "WSO Mk7"
 		(shape bidirectional)
-		(at 135.89 154.94 180)
+		(at 135.89 153.67 180)
 		(fields_autoplaced yes)
 		(effects
@@
 		)
 		(property "Intersheetrefs" "${INTERSHEET_REFS}"
-			(at 123.1455 154.94 0)
+			(at 123.1455 153.67 0)
 			(effects
 				(font
@@
 		(property "Intersheetrefs" "${INTERSHEET_REFS}"
 			(at 184.1945 53.34 0)
-			(effects
-				(font
-					(size 1.27 1.27)
-				)
-				(justify left)
-				(hide yes)
-			)
-		)
-	)
-	(global_label "Vout from Bat reg"
-		(shape input)
-		(at 95.25 40.64 90)
-		(fields_autoplaced yes)
-		(effects
-			(font
-				(size 1.27 1.27)
-			)
-			(justify left)
-		)
-		(property "Intersheetrefs" "${INTERSHEET_REFS}"
-			(at 95.25 20.117 90)
 			(effects
 				(font
@@
 			)
 		)
-		(property "Footprint" "Capacitor_THT:CP_Radial_D5.0mm_P2.50mm"
+		(property "Footprint" "Capacitor_THT:C_Disc_D5.0mm_W2.5mm_P5.00mm"
 			(at 82.55 93.0148 0)
 			(effects
@@
 		(dnp no)
 		(fields_autoplaced yes)
-		(property "Reference" "J7"
+		(property "Reference" "J6"
 			(at 193.04 17.1449 90)
 			(effects
@@
 			(project "highway_wave"
 				(path "/4d93a0f5-0323-4b77-816b-e07a1b9b3cd9/c0d35520-d176-4b46-91a1-98f70e5c8801"
-					(reference "J7")
+					(reference "J6")
 					(unit 1)
 				)
@@
 			)
 		)
-		(property "Footprint" "Capacitor_THT:CP_Radial_D5.0mm_P2.50mm"
+		(property "Footprint" "Capacitor_THT:C_Disc_D5.0mm_W2.5mm_P5.00mm"
 			(at 179.07 142.5448 0)
 			(effects
@@
 			)
 		)
-		(property "Footprint" "Capacitor_THT:CP_Radial_D5.0mm_P2.50mm"
+		(property "Footprint" "Capacitor_THT:C_Disc_D5.0mm_W2.5mm_P5.00mm"
 			(at 82.55 160.3248 0)
 			(effects
@@
 			)
 		)
-		(property "Footprint" "Capacitor_THT:CP_Radial_D5.0mm_P2.50mm"
+		(property "Footprint" "Capacitor_THT:C_Disc_D5.0mm_W2.5mm_P5.00mm"
 			(at 82.55 57.4548 0)
 			(effects
@@
 			)
 		)
-		(property "Footprint" "Capacitor_THT:CP_Radial_D5.0mm_P2.50mm"
+		(property "Footprint" "Capacitor_THT:C_Disc_D5.0mm_W2.5mm_P5.00mm"
 			(at 179.07 75.2348 0)
 			(effects
@@
 			)
 		)
-		(property "Footprint" "Capacitor_THT:CP_Radial_D5.0mm_P2.50mm"
+		(property "Footprint" "Capacitor_THT:C_Disc_D5.0mm_W2.5mm_P5.00mm"
 			(at 179.07 39.6748 0)
 			(effects
@@
 		(dnp no)
 		(fields_autoplaced yes)
-		(property "Reference" "J6"
+		(property "Reference" "J4"
 			(at 120.65 17.1449 90)
 			(effects
@@
 			(project "highway_wave"
 				(path "/4d93a0f5-0323-4b77-816b-e07a1b9b3cd9/c0d35520-d176-4b46-91a1-98f70e5c8801"
-					(reference "J6")
+					(reference "J4")
 					(unit 1)
 				)
@@
 		(dnp no)
 		(fields_autoplaced yes)
-		(property "Reference" "J5"
+		(property "Reference" "J8"
 			(at 64.77 34.9249 90)
 			(effects
@@
 			(project "highway_wave"
 				(path "/4d93a0f5-0323-4b77-816b-e07a1b9b3cd9/c0d35520-d176-4b46-91a1-98f70e5c8801"
-					(reference "J5")
+					(reference "J8")
 					(unit 1)
 				)
@@
 			)
 		)
-		(property "Footprint" "Capacitor_THT:CP_Radial_D5.0mm_P2.50mm"
+		(property "Footprint" "Capacitor_THT:C_Disc_D5.0mm_W2.5mm_P5.00mm"
 			(at 82.55 124.7648 0)
 			(effects
@@
 			)
 		)
-		(property "Footprint" "Capacitor_THT:CP_Radial_D5.0mm_P2.50mm"
+		(property "Footprint" "Capacitor_THT:C_Disc_D5.0mm_W2.5mm_P5.00mm"
 			(at 179.07 106.9848 0)
 			(effects
@@
 		(dnp no)
 		(fields_autoplaced yes)
-		(property "Reference" "J9"
+		(property "Reference" "J10"
 			(at 158.75 17.1449 90)
 			(effects
@@
 			(project "highway_wave"
 				(path "/4d93a0f5-0323-4b77-816b-e07a1b9b3cd9/c0d35520-d176-4b46-91a1-98f70e5c8801"
-					(reference "J9")
+					(reference "J10")
 					(unit 1)
 				)
